File: PCB/GAL_Programmer/GAL_Programmer.kicad_pcb (KiCad board)
At the start: 2 copper layers, 68.6 x 53.3 mm, 8 parts, among them P1 Power, P2 Analog, P3 Digital, P4 Digital, P5 CONN_01X01, P6 CONN_01X01, P7 CONN_01X01, P8 CONN_01X01

Commit message: Se termino el esquematico, falta hacer una revisión a detalle de las conexiones y resistencias que se deben usar, falta agregar capacitores al diseño. Se generó el netlist y se empezo el diseño del PCB
Parts:
- added R1: 4k7, Resistor_THT:R_Axial_DIN0207_L6.3mm_D2.5mm_P7.62mm_Horizontal, F.Cu at (135.9, 85.4)
- added R10: 4k7, Resistor_THT:R_Axial_DIN0207_L6.3mm_D2.5mm_P7.62mm_Horizontal, F.Cu at (135.9, 112.4)
- added R2: 4k7, Resistor_THT:R_Axial_DIN0207_L6.3mm_D2.5mm_P7.62mm_Horizontal, F.Cu at (135.9, 88.4)
- added R3: 4k7, Resistor_THT:R_Axial_DIN0207_L6.3mm_D2.5mm_P7.62mm_Horizontal, F.Cu at (135.9, 91.4)
- added R4: 4k7, Resistor_THT:R_Axial_DIN0207_L6.3mm_D2.5mm_P7.62mm_Horizontal, F.Cu at (135.9, 94.4)
- added R5: 4k7, Resistor_THT:R_Axial_DIN0207_L6.3mm_D2.5mm_P7.62mm_Horizontal, F.Cu at (135.9, 97.4)
- added R6: 4k7, Resistor_THT:R_Axial_DIN0207_L6.3mm_D2.5mm_P7.62mm_Horizontal, F.Cu at (135.9, 100.4)
- added R7: 4k7, Resistor_THT:R_Axial_DIN0207_L6.3mm_D2.5mm_P7.62mm_Horizontal, F.Cu at (135.9, 103.4)
- added R8: 4k7, Resistor_THT:R_Axial_DIN0207_L6.3mm_D2.5mm_P7.62mm_Horizontal, F.Cu at (135.9, 106.4)
- added R9: 4k7, Resistor_THT:R_Axial_DIN0207_L6.3mm_D2.5mm_P7.62mm_Horizontal, F.Cu at (135.9, 109.4)
- added U1: ATF16V8, Package_DIP:DIP-20_W7.62mm_Socket_LongPads, F.Cu at (161.0, 87.9)
- added U2: ATF22V10, Package_DIP:DIP-24_W7.62mm_Socket_LongPads, F.Cu at (156.0, 113.0)
- added U3: MT3608, Socket_Arduino_Uno:MT3608_Module, F.Cu at (123.0, 100.9)
Connections:
- net +3V3 renamed Net-(P1-Pad4)
- P3 pad 7: /11(**/MOSI) -> /11(MOSI)
Routing:
- added copper zone on B.Cu, net GND
- added copper zone on F.Cu, net GND
